File: switchmod.brd (EAGLE design)
At the start: 43 x 43 mm, 38 parts, among them IC2 REG1117, U1 STM32F10XRXT6, X1 USB-MICROB

Commit message: minor board improvements
Parts:
- removed TP1, TP2, TP3, TP5: TEST-POINT3X4, SparkFun-Passives:PAD.03X.04
- added JP5: (no value), adafruit:1X01
- moved C2 2.41 mm to (23.9, 10.2)
- moved C4 1.93 mm to (23.9, 6.10)
- moved R1 0.51 mm to (2.79, 10.9), turned to 90 degrees
- moved R2 0.51 mm to (5.59, 10.9), turned to 90 degrees
- moved R3 0.51 mm to (2.79, 7.37)
- moved R5 0.51 mm to (5.59, 7.37)
- moved Y2 0.14 mm to (27.9, 38.6)
Connections:
- net +3V3: now also JP5.1; no longer JP2.21
- net GND: now also JP2.21
- net N$16: no longer TP1.P$1
- net N$17: no longer TP3.P$1
- net N$18: no longer TP5.P$1
- net N$19: no longer TP2.P$1
- net N$30: no longer R9.2
- net N$32: now also R9.2
Routing:
- net N$18: track 20.6 -> 12.0 mm
- net N$17: track 19.8 -> 11.6 mm
- net N$32: track 17.5 -> 21.3 mm
- net N$19: track 20.9 -> 18.3 mm
- net N$30: track 24.2 -> 22.1 mm
- net GND: track 49.0 -> 47.0 mm, vias 16 -> 17
- net N$16: track 14.7 -> 13.1 mm
- net N$66: track 24.0 -> 22.7 mm
- net N$7: track 8.62 -> 7.74 mm
Other:
- board text added: "BT0"
- board text added: "SwitchMOD dekuNukem 2017"
- board text added: "VIN"
- board text removed: "5V"
- board text removed: "BOOT0"
- board text removed: "MISO"
- board text removed: "MOSI"
- board text removed: "SCK"
- board text removed: "cs"

Commit message: minor board improvements
Parts:
- removed JP5: (no value), adafruit:1X01
- added JP1: JUMPER-PAD-2-NO, SparkFun-Passives:PAD-JUMPER-2-NO_NO_SILK
Connections:
- net +3V3: now also JP1.1; no longer JP5.1
- net N$7: now also JP1.2
Routing:
- net N$7: track 7.74 -> 9.94 mm
Other:
- board text added: "NintenDAC dekuNukem"
- board text removed: "SwitchMOD dekuNukem 2017"
Changed lines of the file:
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@@
 <setting verticaltext="up"/>
 </settings>
-<grid distance="1" unitdist="mil" unit="mil" style="lines" multiple="1" display="no" altdistance="0.025" altunitdist="inch" altunit="inch"/>
+<grid distance="5" unitdist="mil" unit="mil" style="lines" multiple="1" display="no" altdistance="0.025" altunitdist="inch" altunit="inch"/>
 <layers>
 <layer number="1" name="Top" color="4" fill="1" visible="yes" active="yes"/>
@@
 <wire x1="0" y1="43" x2="0" y2="0" width="0" layer="20"/>
 <text x="1.143" y="0.889" size="0.8128" layer="25" rot="R90">REF</text>
-<text x="4.826" y="3.175" size="0.8128" layer="25">0</text>
-<text x="7.366" y="3.175" size="0.8128" layer="25">1</text>
-<text x="9.906" y="3.175" size="0.8128" layer="25">2</text>
-<text x="12.446" y="3.175" size="0.8128" layer="25">3</text>
-<text x="14.986" y="3.175" size="0.8128" layer="25">4</text>
-<text x="17.526" y="3.175" size="0.8128" layer="25">5</text>
-<text x="20.066" y="3.175" size="0.8128" layer="25">6</text>
-<text x="22.606" y="3.175" size="0.8128" layer="25">7</text>
-<text x="24.257" y="3.175" size="0.8128" layer="25">GND</text>
+<text x="4.826" y="3.302" size="0.8128" layer="25">0</text>
+<text x="7.366" y="3.302" size="0.8128" layer="25">1</text>
+<text x="9.906" y="3.302" size="0.8128" layer="25">2</text>
+<text x="12.446" y="3.302" size="0.8128" layer="25">3</text>
+<text x="15.113" y="3.302" size="0.8128" layer="25">4</text>
+<text x="17.526" y="3.302" size="0.8128" layer="25">5</text>
+<text x="20.066" y="3.302" size="0.8128" layer="25">6</text>
+<text x="22.606" y="3.302" size="0.8128" layer="25">7</text>
+<text x="24.257" y="3.302" size="0.8128" layer="25">GND</text>
 <text x="6.858" y="16.764" size="1.016" layer="25">PC9</text>
 <text x="10.033" y="16.764" size="1.016" layer="25">PC8</text>
@@
 <text x="34.6202" y="6.4262" size="0.8128" layer="25">CLK</text>
 <text x="39.7256" y="11.049" size="0.8128" layer="25">3V3</text>
-<text x="40.5892" y="4.5212" size="0.8128" layer="25">GND</text>
+<text x="40.64" y="4.5212" size="0.8128" layer="25">GND</text>
 <text x="39.37" y="41.529" size="0.9144" layer="25">GND</text>
-<text x="1.143" y="3.556" size="0.8128" layer="25" rot="R90">3V3</text>
-<text x="25.908" y="15.3416" size="0.9144" layer="25" rot="R180">SwitchMOD
-dekuNukem 2017</text>
+<text x="24.6888" y="15.4432" size="1.016" layer="25" rot="R180">NintenDAC
+dekuNukem</text>
 </plain>
 <attributes>
@@
 </element>
 <element name="R1" library="SparkFun-Passives" package="0805" value="" x="2.794" y="10.922" smashed="yes" rot="R90">
-<attribute name="NAME" x="1.397" y="10.414" size="0.8128" layer="25" rot="R90"/>
+<attribute name="NAME" x="0.889" y="11.557" size="0.8128" layer="25" rot="R270"/>
 <attribute name="VALUE" x="5.08" y="10.16" size="1.27" layer="27" rot="R90"/>
 </element>
@@
 </element>
 <element name="R2" library="SparkFun-Passives" package="0805" value="" x="5.588" y="10.922" smashed="yes" rot="R90">
-<attribute name="NAME" x="7.493" y="10.414" size="0.8128" layer="25" rot="R90"/>
+<attribute name="NAME" x="6.731" y="11.43" size="0.8128" layer="25" rot="R270"/>
 <attribute name="VALUE" x="7.874" y="10.16" size="1.27" layer="27" rot="R90"/>
 </element>
@@
 </element>
 <element name="R4" library="SparkFun-Passives" package="0805" value="" x="17.145" y="11.684" smashed="yes">
-<attribute name="NAME" x="18.9484" y="11.2776" size="0.8128" layer="25"/>
+<attribute name="NAME" x="18.9484" y="11.4046" size="0.8128" layer="25"/>
 <attribute name="VALUE" x="16.383" y="9.398" size="1.27" layer="27"/>
 </element>
@@
 </element>
 <element name="C10" library="backplane" package="0805" value="" x="17.145" y="9.652" smashed="yes">
-<attribute name="NAME" x="13.6144" y="8.9789" size="0.8128" layer="25"/>
+<attribute name="NAME" x="13.7414" y="9.2329" size="0.8128" layer="25"/>
 <attribute name="VALUE" x="16.129" y="8.255" size="0.4064" layer="27"/>
 </element>
@@
 <attribute name="VALUE" x="19.7612" y="18.1356" size="0.4064" layer="27" rot="R180"/>
 </element>
-<element name="JP5" library="adafruit" package="1X01" value="" x="2.54" y="4.318" smashed="yes">
-<attribute name="VALUE" x="1.27" y="1.143" size="1.27" layer="27"/>
+<element name="JP1" library="SparkFun-Passives" package="PAD-JUMPER-2-NO_NO_SILK" value="JUMPER-PAD-2-NO" x="2.5654" y="4.4196" smashed="yes" rot="R270">
+<attribute name="NAME" x="1.3716" y="3.6132" size="0.8128" layer="25" rot="R90"/>
 </element>
 </elements>
@@
 <wire x1="14.35" y1="7.747" x2="16.1798" y2="7.747" width="0.254" layer="1"/>
 <contactref element="LED2" pad="A"/>
-<contactref element="JP5" pad="1"/>
 <wire x1="18.5928" y1="32.8632" x2="18.5928" y2="32.0548" width="0.2032" layer="1"/>
 <wire x1="18.5928" y1="32.0548" x2="17.907" y2="31.369" width="0.2032" layer="1"/>
@@
 <wire x1="15.9766" y1="29.9212" x2="15.1348" y2="29.9212" width="0.2032" layer="1"/>
 <wire x1="15.1348" y1="29.9212" x2="15.128" y2="29.928" width="0.2032" layer="1"/>
+<contactref element="JP1" pad="1"/>
 </signal>
 <signal name="N$1">
@@
 <wire x1="5.991" y1="3.556" x2="4.318" y2="3.556" width="0.254" layer="1"/>
 <wire x1="4.318" y1="3.556" x2="2.54" y2="1.778" width="0.254" layer="1"/>
+<contactref element="JP1" pad="2"/>
+<wire x1="2.5654" y1="3.9696" x2="2.5654" y2="1.8034" width="0.254" layer="1"/>
+<wire x1="2.5654" y1="1.8034" x2="2.54" y2="1.778" width="0.254" layer="1"/>
 </signal>
 <signal name="N$8">
@@
 <contactref element="JP2" pad="3"/>
 <via x="21.7932" y="18.288" extent="1-16" drill="0.5"/>
-<via x="30.988" y="18.542" extent="1-16" drill="0.5"/>
-<wire x1="30.988" y1="18.542" x2="33.9598" y2="18.542" width="0.254" layer="1"/>
-<wire x1="33.9598" y1="18.542" x2="36.7284" y2="15.7734" width="0.254" layer="1"/>
+<via x="31.0642" y="18.288" extent="1-16" drill="0.5"/>
 <wire x1="36.7284" y1="15.7734" x2="39.3954" y2="15.7734" width="0.254" layer="1"/>
 <wire x1="39.3954" y1="15.7734" x2="40.64" y2="17.018" width="0.254" layer="1"/>
 <wire x1="21.078" y1="21.478" x2="21.078" y2="19.0032" width="0.254" layer="1"/>
 <wire x1="21.078" y1="19.0032" x2="21.7932" y2="18.288" width="0.254" layer="1"/>
-<wire x1="21.7932" y1="18.288" x2="30.734" y2="18.288" width="0.254" layer="16"/>
-<wire x1="30.734" y1="18.288" x2="30.988" y2="18.542" width="0.254" layer="16"/>
+<wire x1="21.7932" y1="18.288" x2="31.0642" y2="18.288" width="0.254" layer="16"/>
+<wire x1="31.0642" y1="18.288" x2="34.2138" y2="18.288" width="0.254" layer="1"/>
+<wire x1="34.2138" y1="18.288" x2="36.7284" y2="15.7734" width="0.254" layer="1"/>
 </signal>
 <signal name="N$33">
@@
 <wire x1="22.078" y1="22.586" x2="22.3012" y2="22.8092" width="0.254" layer="1"/>
 <via x="22.3012" y="22.8092" extent="1-16" drill="0.5"/>
-<via x="30.9626" y="21.336" extent="1-16" drill="0.5"/>
-<wire x1="22.3012" y1="22.8092" x2="29.4894" y2="22.8092" width="0.254" layer="16"/>
-<wire x1="29.4894" y1="22.8092" x2="30.9626" y2="21.336" width="0.254" layer="16"/>
-<wire x1="30.9626" y1="21.336" x2="31.8516" y2="20.447" width="0.254" layer="1"/>
-<wire x1="31.8516" y1="20.447" x2="34.7472" y2="20.447" width="0.254" layer="1"/>
+<via x="30.988" y="20.9042" extent="1-16" drill="0.5"/>
+<wire x1="31.4452" y1="20.447" x2="34.7472" y2="20.447" width="0.254" layer="1"/>
 <wire x1="34.7472" y1="20.447" x2="36.9062" y2="18.288" width="0.254" layer="1"/>
 <wire x1="36.9062" y1="18.288" x2="39.37" y2="18.288" width="0.254" layer="1"/>
 <wire x1="39.37" y1="18.288" x2="40.64" y2="19.558" width="0.254" layer="1"/>
+<wire x1="22.3012" y1="22.8092" x2="29.083" y2="22.8092" width="0.254" layer="16"/>
+<wire x1="29.083" y1="22.8092" x2="30.988" y2="20.9042" width="0.254" layer="16"/>
+<wire x1="30.988" y1="20.9042" x2="31.4452" y2="20.447" width="0.254" layer="1"/>
 </signal>
 <signal name="N$35">
