File: switchmod.sch (EAGLE design)
At the start: 38 parts, among them IC2 REG1117, U1 STM32F10XRXT6, X1 USB-MICROB

Commit message: minor board improvements
Parts:
- removed TP1, TP2, TP3, TP5: TEST-POINT3X4, SparkFun-Passives:TEST-POINT3X4
- added JP5: (no value), adafruit:PINHD-1X1
Connections:
- net +3V3: now also JP5.1; no longer JP2.21
- net GND: now also JP2.21
- net N$16: no longer TP1.1
- net N$17: no longer TP3.1
- net N$18: no longer TP5.1
- net N$19: no longer TP2.1
- net N$30: no longer R9.2
- net N$32: now also R9.2
Other:
- moved on the sheet: R9
Changed lines of the file:
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@@
 <part name="R8" library="SparkFun-Passives" deviceset="RESISTOR" device="0805-RES"/>
 <part name="+3V15" library="backplane" deviceset="+3V3" device=""/>
-<part name="TP1" library="SparkFun-Passives" deviceset="TEST-POINT" device="3X4" value="TEST-POINT3X4"/>
-<part name="TP3" library="SparkFun-Passives" deviceset="TEST-POINT" device="3X4" value="TEST-POINT3X4"/>
-<part name="TP5" library="SparkFun-Passives" deviceset="TEST-POINT" device="3X4" value="TEST-POINT3X4"/>
-<part name="TP2" library="SparkFun-Passives" deviceset="TEST-POINT" device="3X4" value="TEST-POINT3X4"/>
 <part name="LED2" library="backplane" deviceset="LED" device="CHIP-LED0805"/>
 <part name="+3V16" library="backplane" deviceset="+3V3" device=""/>
 <part name="R9" library="SparkFun-Passives" deviceset="RESISTOR" device="0805-RES"/>
-<part name="+3V12" library="backplane" deviceset="+3V3" device=""/>
+<part name="JP5" library="adafruit" deviceset="PINHD-1X1" device=""/>
+<part name="+3V17" library="backplane" deviceset="+3V3" device=""/>
+<part name="GND21" library="backplane" deviceset="GND" device=""/>
 </parts>
 <sheets>
@@
 <instance part="R8" gate="G$1" x="154.94" y="-101.6" rot="R90"/>
 <instance part="+3V15" gate="G$1" x="154.94" y="-93.98"/>
-<instance part="TP1" gate="G$1" x="-27.94" y="-25.4"/>
-<instance part="TP3" gate="G$1" x="-27.94" y="-22.86"/>
-<instance part="TP5" gate="G$1" x="-27.94" y="-20.32"/>
-<instance part="TP2" gate="G$1" x="-27.94" y="-17.78"/>
 <instance part="LED2" gate="G$1" x="-154.94" y="-172.72" rot="R90"/>
 <instance part="+3V16" gate="G$1" x="-160.02" y="-170.18"/>
-<instance part="R9" gate="G$1" x="-139.7" y="-175.26"/>
-<instance part="+3V12" gate="G$1" x="27.94" y="-96.52"/>
+<instance part="R9" gate="G$1" x="-134.62" y="-172.72"/>
+<instance part="JP5" gate="G$1" x="-231.14" y="-48.26"/>
+<instance part="+3V17" gate="G$1" x="-243.84" y="-45.72"/>
+<instance part="GND21" gate="1" x="27.94" y="-101.6"/>
 </instances>
 <busses>
@@
 <wire x1="-157.48" y1="-203.2" x2="-157.48" y2="-195.58" width="0.1524" layer="91"/>
 </segment>
+<segment>
+<pinref part="JP2" gate="A" pin="21"/>
+<wire x1="27.94" y1="-99.06" x2="58.42" y2="-99.06" width="0.1524" layer="91"/>
+<pinref part="GND21" gate="1" pin="GND"/>
+</segment>
 </net>
 <net name="+3V3" class="0">
@@
 </segment>
 <segment>
-<pinref part="+3V12" gate="G$1" pin="+3V3"/>
-<pinref part="JP2" gate="A" pin="21"/>
-<wire x1="27.94" y1="-99.06" x2="58.42" y2="-99.06" width="0.1524" layer="91"/>
+<pinref part="+3V17" gate="G$1" pin="+3V3"/>
+<pinref part="JP5" gate="G$1" pin="1"/>
+<wire x1="-243.84" y1="-48.26" x2="-233.68" y2="-48.26" width="0.1524" layer="91"/>
 </segment>
 </net>
@@
 <wire x1="-50.8" y1="-25.4" x2="-109.22" y2="-22.86" width="0.1524" layer="91"/>
 <pinref part="U1" gate="PORTB_H" pin="PB15"/>
-<pinref part="TP1" gate="G$1" pin="1"/>
-<wire x1="-27.94" y1="-25.4" x2="-50.8" y2="-25.4" width="0.1524" layer="91"/>
-<junction x="-50.8" y="-25.4"/>
 </segment>
 </net>
@@
 <wire x1="-50.8" y1="-22.86" x2="-109.22" y2="-25.4" width="0.1524" layer="91"/>
 <pinref part="U1" gate="PORTB_H" pin="PB14"/>
-<pinref part="TP3" gate="G$1" pin="1"/>
-<wire x1="-50.8" y1="-22.86" x2="-27.94" y2="-22.86" width="0.1524" layer="91"/>
-<junction x="-50.8" y="-22.86"/>
 </segment>
 </net>
@@
 <wire x1="-50.8" y1="-20.32" x2="-109.22" y2="-20.32" width="0.1524" layer="91"/>
 <pinref part="U1" gate="PORTB_H" pin="PB13"/>
-<pinref part="TP5" gate="G$1" pin="1"/>
-<wire x1="-27.94" y1="-20.32" x2="-50.8" y2="-20.32" width="0.1524" layer="91"/>
-<junction x="-50.8" y="-20.32"/>
 </segment>
 </net>
@@
 <wire x1="-68.58" y1="-5.08" x2="-68.58" y2="-17.78" width="0.1524" layer="91"/>
 <junction x="-68.58" y="-17.78"/>
-<pinref part="TP2" gate="G$1" pin="1"/>
-<wire x1="-50.8" y1="-17.78" x2="-27.94" y2="-17.78" width="0.1524" layer="91"/>
-<junction x="-50.8" y="-17.78"/>
 </segment>
 </net>
@@
 <wire x1="-124.46" y1="-172.72" x2="-129.54" y2="-172.72" width="0.1524" layer="91"/>
 <wire x1="-129.54" y1="-172.72" x2="-129.54" y2="-111.76" width="0.1524" layer="91"/>
+<pinref part="R9" gate="G$1" pin="2"/>
+<junction x="-129.54" y="-172.72"/>
 </segment>
 </net>
@@
 <pinref part="JP3" gate="A" pin="4"/>
 <wire x1="-93.98" y1="-111.76" x2="-101.6" y2="-111.76" width="0.1524" layer="91"/>
-<pinref part="R9" gate="G$1" pin="2"/>
-<wire x1="-127" y1="-175.26" x2="-134.62" y2="-175.26" width="0.1524" layer="91"/>
-<junction x="-127" y="-175.26"/>
 </segment>
 </net>
@@
 <pinref part="R9" gate="G$1" pin="1"/>
 <pinref part="LED2" gate="G$1" pin="C"/>
-<wire x1="-144.78" y1="-175.26" x2="-144.78" y2="-172.72" width="0.1524" layer="91"/>
-<wire x1="-144.78" y1="-172.72" x2="-149.86" y2="-172.72" width="0.1524" layer="91"/>
-</segment>
-</net>
+<wire x1="-139.7" y1="-172.72" x2="-149.86" y2="-172.72" width="0.1524" layer="91"/>
+</segment>
+</net>

Commit message: minor board improvements
Parts:
- removed JP5: (no value), adafruit:PINHD-1X1
- added JP1: JUMPER-PAD-2-NO, SparkFun-Passives:JUMPER-PAD-2-NO
Connections:
- net +3V3: now also JP1.1; no longer JP5.1
- net N$7: now also JP1.2
Changed lines of the file:
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@@
 <part name="+3V16" library="backplane" deviceset="+3V3" device=""/>
 <part name="R9" library="SparkFun-Passives" deviceset="RESISTOR" device="0805-RES"/>
-<part name="JP5" library="adafruit" deviceset="PINHD-1X1" device=""/>
-<part name="+3V17" library="backplane" deviceset="+3V3" device=""/>
 <part name="GND21" library="backplane" deviceset="GND" device=""/>
+<part name="JP1" library="SparkFun-Passives" deviceset="JUMPER-PAD-2-NO" device=""/>
+<part name="+3V12" library="backplane" deviceset="+3V3" device=""/>
 </parts>
 <sheets>
@@
 <instance part="+3V16" gate="G$1" x="-160.02" y="-170.18"/>
 <instance part="R9" gate="G$1" x="-134.62" y="-172.72"/>
-<instance part="JP5" gate="G$1" x="-231.14" y="-48.26"/>
-<instance part="+3V17" gate="G$1" x="-243.84" y="-45.72"/>
 <instance part="GND21" gate="1" x="27.94" y="-101.6"/>
+<instance part="JP1" gate="G$1" x="-185.42" y="-5.08"/>
+<instance part="+3V12" gate="G$1" x="-190.5" y="-2.54"/>
 </instances>
 <busses>
@@
 </segment>
 <segment>
-<pinref part="+3V17" gate="G$1" pin="+3V3"/>
-<pinref part="JP5" gate="G$1" pin="1"/>
-<wire x1="-243.84" y1="-48.26" x2="-233.68" y2="-48.26" width="0.1524" layer="91"/>
+<pinref part="JP1" gate="G$1" pin="1"/>
+<pinref part="+3V12" gate="G$1" pin="+3V3"/>
 </segment>
 </net>
@@
 <pinref part="U$2" gate="G$1" pin="1"/>
 <wire x1="-165.1" y1="-5.08" x2="-139.7" y2="-5.08" width="0.1524" layer="91"/>
-</segment>
-</net>
+<pinref part="JP1" gate="G$1" pin="2"/>
+<wire x1="-180.34" y1="-5.08" x2="-165.1" y2="-5.08" width="0.1524" layer="91"/>
+<junction x="-165.1" y="-5.08"/>
+</segment>
+</net>
