File: nintendac.sch (EAGLE design)
At the start: 35 parts, among them IC2 REG1117, U1 STM32F10XRXT6, X1 USB-MICROB

Commit message: added a resistor on ref
Parts:
- removed JP1: JUMPER-PAD-2-NO, SparkFun-Passives:JUMPER-PAD-2-NO
- added R10: (no value), SparkFun-Passives:RESISTOR0805-RES
Connections:
- net +3V3: now also R10.2; no longer JP1.1
- net N$7: now also R10.1; no longer JP1.2
Changed lines of the file:
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@@
 <part name="R9" library="SparkFun-Passives" deviceset="RESISTOR" device="0805-RES"/>
 <part name="GND21" library="backplane" deviceset="GND" device=""/>
-<part name="JP1" library="SparkFun-Passives" deviceset="JUMPER-PAD-2-NO" device=""/>
 <part name="+3V12" library="backplane" deviceset="+3V3" device=""/>
+<part name="R10" library="SparkFun-Passives" deviceset="RESISTOR" device="0805-RES"/>
 </parts>
 <sheets>
@@
 <instance part="R9" gate="G$1" x="-134.62" y="-172.72"/>
 <instance part="GND21" gate="1" x="27.94" y="-101.6"/>
-<instance part="JP1" gate="G$1" x="-185.42" y="-5.08"/>
 <instance part="+3V12" gate="G$1" x="-190.5" y="-2.54"/>
+<instance part="R10" gate="G$1" x="-180.34" y="-5.08" rot="R180"/>
 </instances>
 <busses>
@@
 </segment>
 <segment>
-<pinref part="JP1" gate="G$1" pin="1"/>
 <pinref part="+3V12" gate="G$1" pin="+3V3"/>
+<pinref part="R10" gate="G$1" pin="2"/>
+<wire x1="-190.5" y1="-5.08" x2="-185.42" y2="-5.08" width="0.1524" layer="91"/>
 </segment>
 </net>
@@
 <pinref part="U$2" gate="G$1" pin="1"/>
 <wire x1="-165.1" y1="-5.08" x2="-139.7" y2="-5.08" width="0.1524" layer="91"/>
-<pinref part="JP1" gate="G$1" pin="2"/>
-<wire x1="-180.34" y1="-5.08" x2="-165.1" y2="-5.08" width="0.1524" layer="91"/>
+<pinref part="R10" gate="G$1" pin="1"/>
+<wire x1="-175.26" y1="-5.08" x2="-165.1" y2="-5.08" width="0.1524" layer="91"/>
 <junction x="-165.1" y="-5.08"/>
 </segment>

Commit message: board cleanup
Parts:
- added S2: SWITCH-MOMENTARY-2TURTLE, Adafruit Feather M0 Adalogger:SWITCH-MOMENTARY-2TURTLE
Connections:
- net GND: now also S2.1
- net N$30: now also S2.2
Changed lines of the file:
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@@
 <part name="+3V12" library="backplane" deviceset="+3V3" device=""/>
 <part name="R10" library="SparkFun-Passives" deviceset="RESISTOR" device="0805-RES"/>
+<part name="GND22" library="backplane" deviceset="GND" device=""/>
+<part name="S2" library="Adafruit Feather M0 Adalogger" deviceset="SWITCH-MOMENTARY-2" device="TURTLE"/>
 </parts>
 <sheets>
@@
 <instance part="+3V12" gate="G$1" x="-190.5" y="-2.54"/>
 <instance part="R10" gate="G$1" x="-180.34" y="-5.08" rot="R180"/>
+<instance part="GND22" gate="1" x="-180.34" y="-177.8"/>
+<instance part="S2" gate="G$1" x="-175.26" y="-175.26"/>
 </instances>
 <busses>
@@
 <pinref part="GND21" gate="1" pin="GND"/>
 </segment>
+<segment>
+<pinref part="S2" gate="G$1" pin="1"/>
+<pinref part="GND22" gate="1" pin="GND"/>
+</segment>
 </net>
 <net name="+3V3" class="0">
@@
 <pinref part="JP3" gate="A" pin="4"/>
 <wire x1="-93.98" y1="-111.76" x2="-101.6" y2="-111.76" width="0.1524" layer="91"/>
-</segment>
-</net>
+<wire x1="-127" y1="-175.26" x2="-170.18" y2="-175.26" width="0.1524" layer="91"/>
+<junction x="-127" y="-175.26"/>
+<pinref part="S2" gate="G$1" pin="2"/>
+</segment>
+</net>
