File: mini/nintendac.sch (EAGLE design)
At the start: 30 parts, among them IC1 STM32F10XCXT6, IC2 REG1117, IC3 24C64ST, X1 USB-MICROB

Commit message: updated mini layout
Parts:
- removed C4: (no value), backplane:C-USC1210
- removed C5: (no value), backplane:CAP0805
- removed D1: MBR120, microbuilder:DIODE-SCHOTTKYSOD-123
- removed IC2: REG1117, backplane:REG1117
- added D2: MBR120, microbuilder:DIODE-SCHOTTKYSOD-123
- added R4: (no value), SparkFun-Passives:RESISTOR0805-RES
- added TP1: TEST-POINT3X5, SparkFun-Passives:TEST-POINT3X5
- added U1: (no value), Adafruit Feather M0 Adalogger:VREG_SOT23-5
Connections:
- new net N$31: D2.C, U1.IN
- net +3V3: now also U1.OUT; no longer C5.1, D1.C
- net GND: now also U1.GND; no longer C4.2, C5.2, IC2.GND
- net N$2: now also D2.A, R4.2; no longer C4.1, IC2.VIN
- net N$36: now also R4.1, TP1.1, U1.EN; no longer D1.A, IC2.VOUT
Changed lines of the file:
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@@
 <part name="C2" library="backplane" deviceset="C-US" device="C1210"/>
 <part name="Y1" library="backplane" deviceset="CRYSTAL" device="HC49US"/>
-<part name="IC2" library="backplane" deviceset="REG1117" device=""/>
 <part name="X1" library="backplane" deviceset="USB" device="-MICROB"/>
 <part name="GND2" library="backplane" deviceset="GND" device=""/>
 <part name="GND3" library="backplane" deviceset="GND" device=""/>
 <part name="GND5" library="backplane" deviceset="GND" device=""/>
-<part name="GND6" library="backplane" deviceset="GND" device=""/>
 <part name="+3V3" library="backplane" deviceset="+3V3" device=""/>
 <part name="S1" library="Adafruit Feather M0 Adalogger" deviceset="SWITCH-MOMENTARY-2" device="TURTLE"/>
@@
 <part name="GND7" library="backplane" deviceset="GND" device=""/>
 <part name="GND8" library="backplane" deviceset="GND" device=""/>
-<part name="C4" library="backplane" deviceset="C-US" device="C1210"/>
-<part name="GND9" library="backplane" deviceset="GND" device=""/>
 <part name="GND10" library="backplane" deviceset="GND" device=""/>
-<part name="C5" library="backplane" deviceset="CAP" device="0805"/>
 <part name="C6" library="backplane" deviceset="CAP" device="0805"/>
 <part name="C7" library="backplane" deviceset="CAP" device="0805"/>
@@
 <part name="+3V7" library="backplane" deviceset="+3V3" device=""/>
 <part name="GND15" library="backplane" deviceset="GND" device=""/>
-<part name="D1" library="microbuilder" deviceset="DIODE-SCHOTTKY" device="SOD-123" value="MBR120"/>
 <part name="+3V8" library="backplane" deviceset="+3V3" device=""/>
 <part name="+3V9" library="backplane" deviceset="+3V3" device=""/>
@@
 <part name="S2" library="SparkFun-Retired" deviceset="TAC_SWITCH" device="SMD" value="TAC_SWITCHSMD"/>
 <part name="GND17" library="backplane" deviceset="GND" device=""/>
+<part name="U1" library="Adafruit Feather M0 Adalogger" deviceset="VREG_SOT23-5" device=""/>
+<part name="D2" library="microbuilder" deviceset="DIODE-SCHOTTKY" device="SOD-123" value="MBR120"/>
+<part name="GND6" library="backplane" deviceset="GND" device=""/>
+<part name="R4" library="SparkFun-Passives" deviceset="RESISTOR" device="0805-RES"/>
+<part name="TP1" library="SparkFun-Passives" deviceset="TEST-POINT" device="3X5"/>
 </parts>
 <sheets>
@@
 <instance part="C2" gate="G$1" x="154.94" y="-43.18"/>
 <instance part="Y1" gate="G$1" x="165.1" y="-81.28" rot="R90"/>
-<instance part="IC2" gate="G$1" x="127" y="-38.1"/>
 <instance part="X1" gate="G$1" x="99.06" y="-40.64"/>
 <instance part="GND2" gate="1" x="172.72" y="-109.22"/>
 <instance part="GND3" gate="1" x="-93.98" y="111.76"/>
 <instance part="GND5" gate="1" x="88.9" y="-43.18"/>
-<instance part="GND6" gate="1" x="127" y="-53.34"/>
 <instance part="+3V3" gate="G$1" x="154.94" y="-33.02" rot="MR0"/>
 <instance part="S1" gate="G$1" x="165.1" y="-106.68"/>
@@
 <instance part="GND7" gate="1" x="172.72" y="-93.98"/>
 <instance part="GND8" gate="1" x="190.5" y="-88.9"/>
-<instance part="C4" gate="G$1" x="109.22" y="-40.64"/>
-<instance part="GND9" gate="1" x="109.22" y="-48.26"/>
 <instance part="GND10" gate="1" x="154.94" y="-53.34"/>
-<instance part="C5" gate="G$1" x="10.16" y="101.6"/>
 <instance part="C6" gate="G$1" x="25.4" y="101.6"/>
 <instance part="C7" gate="G$1" x="38.1" y="101.6"/>
@@
 <instance part="+3V7" gate="G$1" x="-78.74" y="-109.22" rot="MR0"/>
 <instance part="GND15" gate="1" x="-68.58" y="-109.22"/>
-<instance part="D1" gate="G$1" x="142.24" y="-38.1"/>
 <instance part="+3V8" gate="G$1" x="27.94" y="-63.5" rot="MR0"/>
 <instance part="+3V9" gate="G$1" x="-45.72" y="-58.42" rot="MR0"/>
@@
 <instance part="S2" gate="S" x="53.34" y="-76.2"/>
 <instance part="GND17" gate="1" x="66.04" y="-78.74"/>
+<instance part="U1" gate="G$1" x="139.7" y="-40.64"/>
+<instance part="D2" gate="G$1" x="121.92" y="-38.1"/>
+<instance part="GND6" gate="1" x="129.54" y="-50.8"/>
+<instance part="R4" gate="G$1" x="116.84" y="-43.18" rot="R90"/>
+<instance part="TP1" gate="G$1" x="119.38" y="-48.26" rot="R90"/>
 </instances>
 <busses>
@@
 </segment>
 <segment>
-<pinref part="IC2" gate="G$1" pin="GND"/>
-<pinref part="GND6" gate="1" pin="GND"/>
-</segment>
-<segment>
 <pinref part="GND2" gate="1" pin="GND"/>
 <pinref part="S1" gate="G$1" pin="2"/>
@@
 <pinref part="C1" gate="G$1" pin="2"/>
 <pinref part="GND8" gate="1" pin="GND"/>
-</segment>
-<segment>
-<pinref part="C4" gate="G$1" pin="2"/>
-<pinref part="GND9" gate="1" pin="GND"/>
 </segment>
 <segment>
@@
 <wire x1="38.1" y1="99.06" x2="25.4" y2="99.06" width="0.1524" layer="91"/>
 <junction x="38.1" y="99.06"/>
-<pinref part="C5" gate="G$1" pin="2"/>
-<wire x1="25.4" y1="99.06" x2="10.16" y2="99.06" width="0.1524" layer="91"/>
-<junction x="25.4" y="99.06"/>
 <pinref part="GND14" gate="1" pin="GND"/>
 <junction x="45.72" y="99.06"/>
@@
 <wire x1="101.6" y1="-58.42" x2="109.22" y2="-58.42" width="0.1524" layer="91"/>
 </segment>
+<segment>
+<pinref part="U1" gate="G$1" pin="GND"/>
+<pinref part="GND6" gate="1" pin="GND"/>
+<wire x1="129.54" y1="-43.18" x2="129.54" y2="-48.26" width="0.1524" layer="91"/>
+</segment>
 </net>
 <net name="+3V3" class="0">
@@
 </segment>
 <segment>
-<pinref part="C5" gate="G$1" pin="1"/>
 <pinref part="C6" gate="G$1" pin="1"/>
-<wire x1="10.16" y1="106.68" x2="25.4" y2="106.68" width="0.1524" layer="91"/>
 <pinref part="C7" gate="G$1" pin="1"/>
 <wire x1="25.4" y1="106.68" x2="38.1" y2="106.68" width="0.1524" layer="91"/>
-<junction x="25.4" y="106.68"/>
 <pinref part="C8" gate="G$1" pin="1"/>
 <wire x1="38.1" y1="106.68" x2="45.72" y2="106.68" width="0.1524" layer="91"/>
@@
 </segment>
 <segment>
-<pinref part="D1" gate="G$1" pin="C"/>
 <pinref part="C2" gate="G$1" pin="1"/>
-<wire x1="144.78" y1="-38.1" x2="154.94" y2="-38.1" width="0.1524" layer="91"/>
-<wire x1="154.94" y1="-38.1" x2="154.94" y2="-40.64" width="0.1524" layer="91"/>
 <pinref part="+3V3" gate="G$1" pin="+3V3"/>
+<wire x1="154.94" y1="-40.64" x2="154.94" y2="-38.1" width="0.1524" layer="91"/>
+<pinref part="U1" gate="G$1" pin="OUT"/>
 <wire x1="154.94" y1="-38.1" x2="154.94" y2="-35.56" width="0.1524" layer="91"/>
+<wire x1="149.86" y1="-38.1" x2="154.94" y2="-38.1" width="0.1524" layer="91"/>
 <junction x="154.94" y="-38.1"/>
 </segment>
@@
 <pinref part="LED2" gate="G$1" pin="C"/>
 <wire x1="-104.14" y1="-132.08" x2="-114.3" y2="-132.08" width="0.1524" layer="91"/>
-</segment>
-</net>
-<net name="N$2" class="0">
-<segment>
-<pinref part="IC2" gate="G$1" pin="VIN"/>
-<pinref part="C4" gate="G$1" pin="1"/>
-<wire x1="109.22" y1="-38.1" x2="114.3" y2="-38.1" width="0.1524" layer="91"/>
-<junction x="109.22" y="-38.1"/>
-<pinref part="X1" gate="G$1" pin="VBUS"/>
-<wire x1="96.52" y1="-38.1" x2="109.22" y2="-38.1" width="0.1524" layer="91"/>
 </segment>
 </net>
@@
 </segment>
 </net>
-<net name="N$36" class="0">
-<segment>
-<pinref part="IC2" gate="G$1" pin="VOUT"/>
-<pinref part="D1" gate="G$1" pin="A"/>
-</segment>
-</net>
 <net name="N$38" class="0">
 <segment>
@@
 </segment>
 </net>
+<net name="N$2" class="0">
+<segment>
+<pinref part="X1" gate="G$1" pin="VBUS"/>
+<wire x1="96.52" y1="-38.1" x2="116.84" y2="-38.1" width="0.1524" layer="91"/>
+<pinref part="D2" gate="G$1" pin="A"/>
+<pinref part="R4" gate="G$1" pin="2"/>
+<wire x1="116.84" y1="-38.1" x2="119.38" y2="-38.1" width="0.1524" layer="91"/>
+<junction x="116.84" y="-38.1"/>
+</segment>
+</net>
+<net name="N$36" class="0">
+<segment>
+<pinref part="R4" gate="G$1" pin="1"/>
+<wire x1="116.84" y1="-48.26" x2="119.38" y2="-48.26" width="0.1524" layer="91"/>
+<wire x1="119.38" y1="-48.26" x2="124.46" y2="-48.26" width="0.1524" layer="91"/>
+<wire x1="124.46" y1="-48.26" x2="124.46" y2="-40.64" width="0.1524" layer="91"/>
+<pinref part="U1" gate="G$1" pin="EN"/>
+<wire x1="124.46" y1="-40.64" x2="129.54" y2="-40.64" width="0.1524" layer="91"/>
+<pinref part="TP1" gate="G$1" pin="1"/>
+<junction x="119.38" y="-48.26"/>
+</segment>
+</net>
+<net name="N$31" class="0">
+<segment>
+<pinref part="U1" gate="G$1" pin="IN"/>
+<pinref part="D2" gate="G$1" pin="C"/>
+<wire x1="124.46" y1="-38.1" x2="129.54" y2="-38.1" width="0.1524" layer="91"/>
+</segment>
+</net>
