File: mini/nintendac.brd (EAGLE design)
At the start: 30 x 45 mm, 30 parts, among them IC1 STM32F10XCXT6, IC2 REG1117, IC3 24C64ST, X1 USB-MICROB

Commit message: updated mini layout
Parts:
- removed C4: (no value), backplane:C1210
- removed C5: (no value), backplane:0805
- removed D1: MBR120, microbuilder:SOD-123
- removed IC2: REG1117, backplane:SOT223
- added D2: MBR120, microbuilder:SOD-123
- added R4: (no value), SparkFun-Passives:0805
- added TP1: TEST-POINT3X5, SparkFun-Passives:PAD.03X.05
- added U1: (no value), Adafruit Feather M0 Adalogger:SOT23-5
- moved C2 5.33 mm to (23.2, 39.5), turned to 180 degrees
- moved R2 5.29 mm to (21.0, 22.5), turned to 45 degrees
- moved U$2 4.01 mm to (24.3, 27.1)
- moved X1 3.49 mm to (15.8, 40.2)
- moved JP1 2.62 mm to (5.63, 39.9)
- moved IC3 2.50 mm to (20.6, 27.8)
- moved LED2 2.38 mm to (8.39, 1.57), turned to 90 degrees
- moved R3 2.37 mm to (17.9, 25.2)
- moved PWR 2.28 mm to (4.16, 26.2)
- moved C1 1.99 mm to (17.8, 5.92)
- moved C3 1.99 mm to (17.8, 9.22)
- moved C8 1.99 mm to (17.3, 14.9)
- moved IC1 1.99 mm to (13.0, 20.1)
- moved R7 1.99 mm to (6.26, 24.9)
- moved R8 1.99 mm to (20.7, 9.02)
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Connections:
- new net N$31: D2.C, U1.1
- net +3V3: now also U1.5; no longer C5.1, D1.C
- net GND: now also U1.2; no longer C4.2, C5.2, IC2.1
- net N$2: now also D2.A, R4.2; no longer C4.1, IC2.3
- net N$36: now also R4.1, TP1.P$1, U1.3; no longer D1.A, IC2.2
Routing:
- net +3V3: track 168.8 -> 55.2 mm
- net GND: track 56.8 -> 42.5 mm, vias 13 -> 12
- net N$36: track 2.67 -> 11.0 mm
- net N$9: track 31.6 -> 26.3 mm
- net N$2: track 10.1 -> 5.56 mm
- net N$31: track 0.00 -> 3.88 mm
- net N$8: track 20.3 -> 17.1 mm
- net N$7: track 17.8 -> 15.1 mm
- net N$4: track 17.7 -> 15.1 mm
- net N$43: track 20.3 -> 17.9 mm
- net N$39: track 17.3 -> 15.1 mm
- net N$3: track 14.9 -> 12.8 mm
- net N$38: track 14.9 -> 12.9 mm
- net N$14: track 10.4 -> 8.34 mm
- net N$1: track 20.4 -> 18.4 mm
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Other:
- board size 30 x 45 mm -> 26 x 42 mm
- board text added: "C13"
- board text removed: "PC13"

Commit message: board cleanup
Routing:
- net +3V3: track 55.2 -> 54.3 mm
Changed lines of the file:
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@@
 <wire x1="14.2654" y1="16.5608" x2="14.2654" y2="15.5822" width="0.2032" layer="1"/>
 <wire x1="14.2654" y1="15.5822" x2="14.2594" y2="15.5762" width="0.2032" layer="1"/>
-<wire x1="19.0406" y1="15.7226" x2="18.1008" y2="15.7226" width="0.2032" layer="1"/>
-<wire x1="18.1008" y1="15.7226" x2="17.3134" y2="15.7226" width="0.2032" layer="1"/>
 <wire x1="23.7142" y1="11.0744" x2="21.5552" y2="13.2334" width="0.2032" layer="1"/>
 <wire x1="21.5552" y1="13.2334" x2="20.5138" y2="13.2334" width="0.2032" layer="1"/>
-<wire x1="20.5138" y1="13.2334" x2="18.1008" y2="15.6464" width="0.2032" layer="1"/>
-<wire x1="18.1008" y1="15.6464" x2="18.1008" y2="15.7226" width="0.2032" layer="1"/>
+<wire x1="20.5138" y1="13.2334" x2="17.9882" y2="15.759" width="0.2032" layer="1"/>
 <contactref element="JP1" pad="4"/>
 <contactref element="U1" pad="5"/>
@@
 <wire x1="23.4696" y1="27.0764" x2="24.8666" y2="27.0764" width="0.2032" layer="1"/>
 <wire x1="24.8666" y1="27.0764" x2="25.4508" y2="26.4922" width="0.2032" layer="1"/>
+<wire x1="17.9882" y1="15.759" x2="17.2626" y2="15.759" width="0.2032" layer="1"/>
 <wire x1="19.7924" y1="35.5393" x2="19.7772" y2="35.6108" width="0" layer="19" extent="1-1"/>
 </signal>

Commit message: board cleanup
Parts:
- moved PWR 0.80 mm to (4.92, 26.0)
- moved R7 0.51 mm to (6.77, 24.9)
Routing:
- net GND: track 42.5 -> 46.7 mm
Other:
- board text added: "PA8"
- board text added: "PC 13"
- board text added: "PC13"
- board text added: "PWR"
- board text removed: "C13"

Commit message: board cleanup
Parts:
- moved Y1 0.38 mm to (14.3, 7.97)
Other:
- board text added: "2017"
- board text added: "A0"
- board text added: "A1"
- board text added: "A10"
- board text added: "A15"
- board text added: "A2"
- board text added: "A3"
- board text added: "A4"
- board text added: "A5"
- board text added: "A6"
- board text added: "A7"
- board text added: "A8"
- board text added: "A9"
- board text added: "B0"
- board text added: "B1"
- board text added: "B10"
- board text added: "B11"
- board text added: "B12"
- board text added: "B13"
- board text added: "B14"
- board text added: "B15"
- board text added: "B2"
- board text added: "B3"
- board text added: "B4"
- board text added: "B5"
- board text added: "B6"
- board text added: "B7"
- board text added: "B8"
- board text added: "B9"
- board text added: "BT0"
- board text added: "C13"
- board text added: "G"
- board text added: "NintenDAC mini"
- board text added: "RST"
- board text added: "dekuNukem"
- board text removed: "PC 13"

Commit message: board cleanup
Changed lines of the file:
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@@
 <text x="2.7686" y="4.81" size="0.8128" layer="25" rot="R270">VB</text>
 <text x="0.8288" y="37.3126" size="0.8128" layer="25">3V3</text>
-<text x="3.4958" y="37.3126" size="0.8128" layer="25">CLK</text>
+<text x="3.2418" y="37.3126" size="0.8128" layer="25">CLK</text>
 <text x="5.9088" y="37.3126" size="0.8128" layer="25">DIO</text>
 <text x="8.3218" y="37.3126" size="0.8128" layer="25">GND</text>
@@
 <text x="2.7432" y="8.5852" size="0.8128" layer="25" distance="10" rot="R270">B8</text>
 <text x="2.7432" y="10.9982" size="0.8128" layer="25" distance="10" rot="R270">BT0</text>
-<text x="2.7432" y="12.6492" size="0.8128" layer="25" distance="10" rot="R270">B7</text>
+<text x="2.7432" y="12.7762" size="0.8128" layer="25" distance="10" rot="R270">B7</text>
 <text x="2.7432" y="14.6812" size="0.8128" layer="25" distance="10" rot="R270">B6</text>
 <text x="2.7432" y="16.7132" size="0.8128" layer="25" distance="10" rot="R270">B5</text>
-<text x="2.7432" y="18.6182" size="0.8128" layer="25" distance="10" rot="R270">B4</text>
+<text x="2.7432" y="18.7452" size="0.8128" layer="25" distance="10" rot="R270">B4</text>
 <text x="2.7432" y="20.6502" size="0.8128" layer="25" distance="10" rot="R270">B3</text>
 <text x="2.7432" y="22.9362" size="0.8128" layer="25" distance="10" rot="R270">A15</text>
 <text x="2.7432" y="25.0952" size="0.8128" layer="25" distance="10" rot="R270">A10</text>
-<text x="2.7432" y="26.6192" size="0.8128" layer="25" distance="10" rot="R270">A9</text>
+<text x="2.7432" y="26.7462" size="0.8128" layer="25" distance="10" rot="R270">A9</text>
 <text x="2.7432" y="28.6512" size="0.8128" layer="25" distance="10" rot="R270">A8</text>
 <text x="2.7432" y="30.9372" size="0.8128" layer="25" distance="10" rot="R270">B15</text>
 <text x="2.7432" y="33.0962" size="0.8128" layer="25" distance="10" rot="R270">B14</text>
-<text x="2.7432" y="34.3662" size="0.8128" layer="25" distance="10" rot="R270">G</text>
+<text x="2.7432" y="34.4932" size="0.8128" layer="25" distance="10" rot="R270">G</text>
 <text x="2.7432" y="37.0332" size="0.8128" layer="25" distance="10" rot="R270">3V3</text>
-<text x="23.3934" y="1.54" size="0.8128" layer="25" rot="R90">G</text>
+<text x="23.3934" y="1.667" size="0.8128" layer="25" rot="R90">G</text>
 <text x="23.3934" y="3.064" size="0.8128" layer="25" rot="R90">RST</text>
 <text x="23.3934" y="5.477" size="0.8128" layer="25" rot="R90">A0</text>
@@
 <text x="23.3934" y="19.447" size="0.8128" layer="25" rot="R90">A7</text>
 <text x="23.3934" y="21.479" size="0.8128" layer="25" rot="R90">B0</text>
-<text x="23.3934" y="23.384" size="0.8128" layer="25" rot="R90">B1</text>
+<text x="23.3934" y="23.511" size="0.8128" layer="25" rot="R90">B1</text>
 <text x="23.3934" y="25.416" size="0.8128" layer="25" rot="R90">B2</text>
 <text x="23.3934" y="27.067" size="0.8128" layer="25" rot="R90">B10</text>
@@
 <wire x1="24.8666" y1="27.0764" x2="25.4508" y2="26.4922" width="0.2032" layer="1"/>
 <wire x1="17.9882" y1="15.759" x2="17.2626" y2="15.759" width="0.2032" layer="1"/>
+<wire x1="21.5904" y1="24.8372" x2="21.5904" y2="23.1831875" width="0.2032" layer="1"/>
 <wire x1="19.7924" y1="35.5393" x2="19.7772" y2="35.6108" width="0" layer="19" extent="1-1"/>
-<wire x1="21.5904" y1="24.8372" x2="21.5904" y2="23.1831875" width="0.2032" layer="1"/>
 </signal>
 <signal name="N$1">
