File: NintenDAC/nintendac.sch (EAGLE design)
At the start: 36 parts, among them IC2 REG1117, U1 STM32F10XRXT6, X1 USB-MICROB

Commit message: board cleanup
Parts:
- removed C4: (no value), backplane:C-USC1210
- removed IC2: REG1117, backplane:REG1117
- added D1, D2: (no value), nintendac_mini:DIODE-SCHOTTKYSOD-123
- added U2: (no value), nintendac_mini:VREG_SOT23-5
Connections:
- new net N$2: D1.C, D2.C, U2.EN, U2.IN
- net +3V3: now also U2.OUT; no longer IC2.VOUT
- net GND: now also U2.GND; no longer C4.2, IC2.GND
- net N$58: now also D2.A, X1.VBUS
- net N$66: now also D1.A; no longer C4.1, IC2.VIN, X1.VBUS
Other:
- moved on the sheet: C2
Changed lines of the file:
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@@
 <part name="GND1" library="backplane" deviceset="GND" device=""/>
 <part name="R1" library="SparkFun-Passives" deviceset="RESISTOR" device="0805-RES"/>
-<part name="IC2" library="backplane" deviceset="REG1117" device=""/>
 <part name="X1" library="backplane" deviceset="USB" device="-MICROB"/>
 <part name="GND2" library="backplane" deviceset="GND" device=""/>
@@
 <part name="+3V2" library="backplane" deviceset="+3V3" device=""/>
 <part name="GND5" library="backplane" deviceset="GND" device=""/>
-<part name="GND6" library="backplane" deviceset="GND" device=""/>
 <part name="+3V3" library="backplane" deviceset="+3V3" device=""/>
 <part name="S1" library="Adafruit Feather M0 Adalogger" deviceset="SWITCH-MOMENTARY-2" device="TURTLE"/>
@@
 <part name="GND7" library="backplane" deviceset="GND" device=""/>
 <part name="GND8" library="backplane" deviceset="GND" device=""/>
-<part name="C4" library="backplane" deviceset="C-US" device="C1210"/>
-<part name="GND9" library="backplane" deviceset="GND" device=""/>
 <part name="GND10" library="backplane" deviceset="GND" device=""/>
 <part name="GND11" library="backplane" deviceset="GND" device=""/>
@@
 <part name="GND22" library="backplane" deviceset="GND" device=""/>
 <part name="S2" library="Adafruit Feather M0 Adalogger" deviceset="SWITCH-MOMENTARY-2" device="TURTLE"/>
+<part name="D1" library="nintendac_mini" deviceset="DIODE-SCHOTTKY" device="SOD-123"/>
+<part name="D2" library="nintendac_mini" deviceset="DIODE-SCHOTTKY" device="SOD-123"/>
+<part name="U2" library="nintendac_mini" deviceset="VREG_SOT23-5" device=""/>
+<part name="GND6" library="backplane" deviceset="GND" device=""/>
 </parts>
 <sheets>
@@
 <instance part="+3V1" gate="G$1" x="-93.98" y="162.56"/>
 <instance part="C1" gate="G$1" x="190.5" y="-83.82"/>
-<instance part="C2" gate="G$1" x="142.24" y="-40.64"/>
+<instance part="C2" gate="G$1" x="175.26" y="-40.64"/>
 <instance part="Y1" gate="G$1" x="165.1" y="-81.28" rot="R90"/>
 <instance part="GND1" gate="1" x="-7.62" y="43.18"/>
 <instance part="R1" gate="G$1" x="-91.44" y="0" rot="R90"/>
-<instance part="IC2" gate="G$1" x="127" y="-38.1"/>
 <instance part="X1" gate="G$1" x="99.06" y="-40.64"/>
 <instance part="GND2" gate="1" x="172.72" y="-109.22"/>
@@
 <instance part="+3V2" gate="G$1" x="157.48" y="-134.62"/>
 <instance part="GND5" gate="1" x="88.9" y="-43.18"/>
-<instance part="GND6" gate="1" x="127" y="-53.34"/>
-<instance part="+3V3" gate="G$1" x="147.32" y="-35.56"/>
+<instance part="+3V3" gate="G$1" x="185.42" y="-35.56"/>
 <instance part="S1" gate="G$1" x="165.1" y="-106.68"/>
 <instance part="JP2" gate="A" x="60.96" y="-86.36"/>
@@
 <instance part="GND7" gate="1" x="172.72" y="-93.98"/>
 <instance part="GND8" gate="1" x="190.5" y="-88.9"/>
-<instance part="C4" gate="G$1" x="109.22" y="-40.64"/>
-<instance part="GND9" gate="1" x="109.22" y="-48.26"/>
-<instance part="GND10" gate="1" x="142.24" y="-48.26"/>
+<instance part="GND10" gate="1" x="175.26" y="-48.26"/>
 <instance part="GND11" gate="1" x="-157.48" y="-30.48"/>
 <instance part="+3V4" gate="G$1" x="-124.46" y="-35.56"/>
@@
 <instance part="GND22" gate="1" x="-180.34" y="-177.8"/>
 <instance part="S2" gate="G$1" x="-175.26" y="-175.26"/>
+<instance part="D1" gate="G$1" x="124.46" y="-43.18"/>
+<instance part="D2" gate="G$1" x="124.46" y="-38.1"/>
+<instance part="U2" gate="G$1" x="152.4" y="-40.64"/>
+<instance part="GND6" gate="1" x="142.24" y="-45.72"/>
 </instances>
 <busses>
@@
 </segment>
 <segment>
-<pinref part="IC2" gate="G$1" pin="GND"/>
-<pinref part="GND6" gate="1" pin="GND"/>
-</segment>
-<segment>
 <pinref part="GND2" gate="1" pin="GND"/>
 <pinref part="S1" gate="G$1" pin="2"/>
@@
 <pinref part="C1" gate="G$1" pin="2"/>
 <pinref part="GND8" gate="1" pin="GND"/>
-</segment>
-<segment>
-<pinref part="C4" gate="G$1" pin="2"/>
-<pinref part="GND9" gate="1" pin="GND"/>
 </segment>
 <segment>
@@
 <pinref part="GND22" gate="1" pin="GND"/>
 </segment>
+<segment>
+<pinref part="U2" gate="G$1" pin="GND"/>
+<pinref part="GND6" gate="1" pin="GND"/>
+</segment>
 </net>
 <net name="+3V3" class="0">
@@
 </segment>
 <segment>
-<pinref part="IC2" gate="G$1" pin="VOUT"/>
 <pinref part="+3V3" gate="G$1" pin="+3V3"/>
-<wire x1="147.32" y1="-38.1" x2="142.24" y2="-38.1" width="0.1524" layer="91"/>
+<wire x1="185.42" y1="-38.1" x2="175.26" y2="-38.1" width="0.1524" layer="91"/>
 <pinref part="C2" gate="G$1" pin="1"/>
-<wire x1="142.24" y1="-38.1" x2="139.7" y2="-38.1" width="0.1524" layer="91"/>
-<junction x="142.24" y="-38.1"/>
+<pinref part="U2" gate="G$1" pin="OUT"/>
+<wire x1="162.56" y1="-38.1" x2="175.26" y2="-38.1" width="0.1524" layer="91"/>
+<junction x="175.26" y="-38.1"/>
 </segment>
 <segment>
@@
 <pinref part="JP2" gate="A" pin="13"/>
 <wire x1="43.18" y1="-88.9" x2="58.42" y2="-88.9" width="0.1524" layer="91"/>
+<pinref part="D2" gate="G$1" pin="A"/>
+<pinref part="X1" gate="G$1" pin="VBUS"/>
+<wire x1="96.52" y1="-38.1" x2="114.3" y2="-38.1" width="0.1524" layer="91"/>
+<wire x1="114.3" y1="-38.1" x2="121.92" y2="-38.1" width="0.1524" layer="91"/>
+<wire x1="71.12" y1="-134.62" x2="114.3" y2="-134.62" width="0.1524" layer="91"/>
+<wire x1="114.3" y1="-134.62" x2="114.3" y2="-38.1" width="0.1524" layer="91"/>
+<junction x="71.12" y="-134.62"/>
+<junction x="114.3" y="-38.1"/>
 </segment>
 </net>
@@
 </segment>
 </net>
+<net name="N$2" class="0">
+<segment>
+<pinref part="D2" gate="G$1" pin="C"/>
+<pinref part="U2" gate="G$1" pin="IN"/>
+<wire x1="127" y1="-38.1" x2="134.62" y2="-38.1" width="0.1524" layer="91"/>
+<pinref part="D1" gate="G$1" pin="C"/>
+<wire x1="134.62" y1="-38.1" x2="142.24" y2="-38.1" width="0.1524" layer="91"/>
+<wire x1="127" y1="-43.18" x2="134.62" y2="-43.18" width="0.1524" layer="91"/>
+<wire x1="134.62" y1="-43.18" x2="134.62" y2="-40.64" width="0.1524" layer="91"/>
+<junction x="134.62" y="-38.1"/>
+<pinref part="U2" gate="G$1" pin="EN"/>
+<wire x1="134.62" y1="-40.64" x2="134.62" y2="-38.1" width="0.1524" layer="91"/>
+<wire x1="142.24" y1="-40.64" x2="134.62" y2="-40.64" width="0.1524" layer="91"/>
+<junction x="134.62" y="-40.64"/>
+</segment>
+</net>
 <net name="N$66" class="0">
 <segment>
 <pinref part="JP2" gate="A" pin="2"/>
-<pinref part="X1" gate="G$1" pin="VBUS"/>
-<pinref part="IC2" gate="G$1" pin="VIN"/>
-<wire x1="96.52" y1="-38.1" x2="106.68" y2="-38.1" width="0.1524" layer="91"/>
-<pinref part="C4" gate="G$1" pin="1"/>
-<wire x1="106.68" y1="-38.1" x2="109.22" y2="-38.1" width="0.1524" layer="91"/>
-<wire x1="109.22" y1="-38.1" x2="114.3" y2="-38.1" width="0.1524" layer="91"/>
-<junction x="109.22" y="-38.1"/>
-<wire x1="66.04" y1="-73.66" x2="106.68" y2="-73.66" width="0.1524" layer="91"/>
-<wire x1="106.68" y1="-73.66" x2="106.68" y2="-38.1" width="0.1524" layer="91"/>
-<junction x="106.68" y="-38.1"/>
-</segment>
-</net>
+<pinref part="D1" gate="G$1" pin="A"/>
+<wire x1="66.04" y1="-73.66" x2="121.92" y2="-73.66" width="0.1524" layer="91"/>
+<wire x1="121.92" y1="-73.66" x2="121.92" y2="-43.18" width="0.1524" layer="91"/>
+</segment>
+</net>

Commit message: added EEPROM
Parts:
- added IC1: 24LC64ST, nintendac_mini:24LC64ST
- added R11, R12: (no value), SparkFun-Passives:RESISTOR0805-RES
- added TP1: TEST-POINT3X5, SparkFun-Connectors:TEST-POINT3X5
Connections:
- new net N$67: IC1.SCL, R11.1, U1PORTB_H.PB10
- new net N$68: IC1.SDA, R12.1, U1PORTB_H.PB11
- new net N$69: TP1.1, U1PORTB_L.PB2
- net +3V3: now also IC1.VCC, R11.2, R12.2
- net GND: now also IC1.A0, IC1.A1, IC1.A2, IC1.GND, IC1.WP
- net LDAC: no longer U1PORTB_L.PB2
- net N$20: no longer U1PORTB_H.PB11
- net N$21: no longer U1PORTB_H.PB10
Changed lines of the file:
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@@
 <part name="C2" library="backplane" deviceset="C-US" device="C1210"/>
 <part name="Y1" library="backplane" deviceset="CRYSTAL" device="HC49US"/>
-<part name="GND1" library="backplane" deviceset="GND" device=""/>
 <part name="R1" library="SparkFun-Passives" deviceset="RESISTOR" device="0805-RES"/>
 <part name="X1" library="backplane" deviceset="USB" device="-MICROB"/>
@@
 <part name="U2" library="nintendac_mini" deviceset="VREG_SOT23-5" device=""/>
 <part name="GND6" library="backplane" deviceset="GND" device=""/>
+<part name="IC1" library="nintendac_mini" deviceset="24*" device="ST" technology="LC64"/>
+<part name="R11" library="SparkFun-Passives" deviceset="RESISTOR" device="0805-RES"/>
+<part name="R12" library="SparkFun-Passives" deviceset="RESISTOR" device="0805-RES"/>
+<part name="+3V17" library="backplane" deviceset="+3V3" device=""/>
+<part name="+3V18" library="backplane" deviceset="+3V3" device=""/>
+<part name="GND9" library="backplane" deviceset="GND" device=""/>
+<part name="GND23" library="backplane" deviceset="GND" device=""/>
+<part name="+3V19" library="backplane" deviceset="+3V3" device=""/>
+<part name="TP1" library="SparkFun-Connectors" deviceset="TEST-POINT" device="3X5"/>
 </parts>
 <sheets>
@@
 <instance part="C2" gate="G$1" x="175.26" y="-40.64"/>
 <instance part="Y1" gate="G$1" x="165.1" y="-81.28" rot="R90"/>
-<instance part="GND1" gate="1" x="-7.62" y="43.18"/>
 <instance part="R1" gate="G$1" x="-91.44" y="0" rot="R90"/>
 <instance part="X1" gate="G$1" x="99.06" y="-40.64"/>
@@
 <instance part="U2" gate="G$1" x="152.4" y="-40.64"/>
 <instance part="GND6" gate="1" x="142.24" y="-45.72"/>
+<instance part="IC1" gate="G$1" x="-38.1" y="40.64"/>
+<instance part="R11" gate="G$1" x="-55.88" y="53.34" rot="R90"/>
+<instance part="R12" gate="G$1" x="-17.78" y="45.72" rot="R90"/>
+<instance part="+3V17" gate="G$1" x="-17.78" y="53.34"/>
+<instance part="+3V18" gate="G$1" x="-55.88" y="60.96"/>
+<instance part="GND9" gate="1" x="-30.48" y="27.94"/>
+<instance part="GND23" gate="1" x="-53.34" y="30.48"/>
+<instance part="+3V19" gate="G$1" x="-30.48" y="55.88"/>
+<instance part="TP1" gate="G$1" x="93.98" y="-127"/>
 </instances>
 <busses>
@@
 <pinref part="GND6" gate="1" pin="GND"/>
 </segment>
+<segment>
+<pinref part="IC1" gate="G$1" pin="GND"/>
+<pinref part="GND9" gate="1" pin="GND"/>
+</segment>
+<segment>
+<pinref part="GND23" gate="1" pin="GND"/>
+<pinref part="IC1" gate="G$1" pin="WP"/>
+<wire x1="-53.34" y1="33.02" x2="-53.34" y2="35.56" width="0.1524" layer="91"/>
+<wire x1="-53.34" y1="35.56" x2="-53.34" y2="38.1" width="0.1524" layer="91"/>
+<wire x1="-53.34" y1="38.1" x2="-53.34" y2="40.64" width="0.1524" layer="91"/>
+<wire x1="-53.34" y1="40.64" x2="-53.34" y2="45.72" width="0.1524" layer="91"/>
+<wire x1="-53.34" y1="45.72" x2="-50.8" y2="45.72" width="0.1524" layer="91"/>
+<pinref part="IC1" gate="G$1" pin="A2"/>
+<wire x1="-50.8" y1="40.64" x2="-53.34" y2="40.64" width="0.1524" layer="91"/>
+<junction x="-53.34" y="40.64"/>
+<pinref part="IC1" gate="G$1" pin="A1"/>
+<wire x1="-50.8" y1="38.1" x2="-53.34" y2="38.1" width="0.1524" layer="91"/>
+<junction x="-53.34" y="38.1"/>
+<pinref part="IC1" gate="G$1" pin="A0"/>
+<wire x1="-50.8" y1="35.56" x2="-53.34" y2="35.56" width="0.1524" layer="91"/>
+<junction x="-53.34" y="35.56"/>
+</segment>
 </net>
 <net name="+3V3" class="0">
@@
 <wire x1="-190.5" y1="-5.08" x2="-185.42" y2="-5.08" width="0.1524" layer="91"/>
 </segment>
+<segment>
+<pinref part="R12" gate="G$1" pin="2"/>
+<pinref part="+3V17" gate="G$1" pin="+3V3"/>
+</segment>
+<segment>
+<pinref part="R11" gate="G$1" pin="2"/>
+<pinref part="+3V18" gate="G$1" pin="+3V3"/>
+</segment>
+<segment>
+<pinref part="IC1" gate="G$1" pin="VCC"/>
+<pinref part="+3V19" gate="G$1" pin="+3V3"/>
+</segment>
 </net>
 <net name="N$1" class="0">
@@
 <segment>
 <pinref part="U$1" gate="G$1" pin="IRQ"/>
-<wire x1="-50.8" y1="-15.24" x2="-60.96" y2="-15.24" width="0.1524" layer="91"/>
-<pinref part="U1" gate="PORTB_H" pin="PB11"/>
 <pinref part="R5" gate="G$1" pin="1"/>
 <wire x1="-60.96" y1="-15.24" x2="-109.22" y2="-15.24" width="0.1524" layer="91"/>
 <wire x1="-60.96" y1="-5.08" x2="-60.96" y2="-15.24" width="0.1524" layer="91"/>
-<junction x="-60.96" y="-15.24"/>
 </segment>
 </net>
@@
 <pinref part="U$1" gate="G$1" pin="CLR"/>
 <wire x1="-109.22" y1="-12.7" x2="-76.2" y2="-12.7" width="0.1524" layer="91"/>
-<pinref part="U1" gate="PORTB_H" pin="PB10"/>
 <pinref part="R3" gate="G$1" pin="1"/>
-<wire x1="-76.2" y1="-12.7" x2="-50.8" y2="-12.7" width="0.1524" layer="91"/>
 <wire x1="-76.2" y1="-5.08" x2="-76.2" y2="-12.7" width="0.1524" layer="91"/>
-<junction x="-76.2" y="-12.7"/>
 </segment>
 </net>
@@
 </net>
 <net name="LDAC" class="0">
-<segment>
-<pinref part="U1" gate="PORTB_L" pin="PB2"/>
-<wire x1="71.12" y1="-127" x2="91.44" y2="-127" width="0.1524" layer="91"/>
-<label x="86.36" y="-127" size="1.778" layer="95"/>
-</segment>
 <segment>
 <pinref part="R2" gate="G$1" pin="1"/>
@@
 </segment>
 </net>
+<net name="N$67" class="0">
+<segment>
+<pinref part="IC1" gate="G$1" pin="SCL"/>
+<pinref part="R11" gate="G$1" pin="1"/>
+<wire x1="-50.8" y1="48.26" x2="-55.88" y2="48.26" width="0.1524" layer="91"/>
+<pinref part="U1" gate="PORTB_H" pin="PB10"/>
+<wire x1="-55.88" y1="48.26" x2="-55.88" y2="-12.7" width="0.1524" layer="91"/>
+<wire x1="-55.88" y1="-12.7" x2="-50.8" y2="-12.7" width="0.1524" layer="91"/>
+<junction x="-55.88" y="48.26"/>
+</segment>
+</net>
+<net name="N$68" class="0">
+<segment>
+<pinref part="IC1" gate="G$1" pin="SDA"/>
+<pinref part="R12" gate="G$1" pin="1"/>
+<wire x1="-22.86" y1="40.64" x2="-17.78" y2="40.64" width="0.1524" layer="91"/>
+<pinref part="U1" gate="PORTB_H" pin="PB11"/>
+<wire x1="-17.78" y1="40.64" x2="-17.78" y2="-15.24" width="0.1524" layer="91"/>
+<wire x1="-17.78" y1="-15.24" x2="-50.8" y2="-15.24" width="0.1524" layer="91"/>
+<junction x="-17.78" y="40.64"/>
+</segment>
+</net>
+<net name="N$69" class="0">
+<segment>
+<pinref part="TP1" gate="G$1" pin="1"/>
+<pinref part="U1" gate="PORTB_L" pin="PB2"/>
+<wire x1="93.98" y1="-127" x2="71.12" y2="-127" width="0.1524" layer="91"/>
+</segment>
+</net>

Commit message: removed wkup from headers
Parts:
- removed TP1: TEST-POINT3X5, SparkFun-Connectors:TEST-POINT3X5
- added R13: (no value), SparkFun-Passives:RESISTOR0805-RES
Connections:
- net GND: now also R13.1
- net N$58: now also R13.2; no longer JP2.13
- net N$69: now also JP2.13; no longer TP1.1
Changed lines of the file:
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@@
 <part name="GND23" library="backplane" deviceset="GND" device=""/>
 <part name="+3V19" library="backplane" deviceset="+3V3" device=""/>
-<part name="TP1" library="SparkFun-Connectors" deviceset="TEST-POINT" device="3X5"/>
+<part name="R13" library="SparkFun-Passives" deviceset="RESISTOR" device="0805-RES"/>
+<part name="GND1" library="backplane" deviceset="GND" device=""/>
 </parts>
 <sheets>
@@
 <instance part="GND23" gate="1" x="-53.34" y="30.48"/>
 <instance part="+3V19" gate="G$1" x="-30.48" y="55.88"/>
-<instance part="TP1" gate="G$1" x="93.98" y="-127"/>
+<instance part="R13" gate="G$1" x="109.22" y="-43.18" rot="R90"/>
+<instance part="GND1" gate="1" x="109.22" y="-50.8"/>
 </instances>
 <busses>
@@
 <junction x="-53.34" y="35.56"/>
 </segment>
+<segment>
+<pinref part="R13" gate="G$1" pin="1"/>
+<pinref part="GND1" gate="1" pin="GND"/>
+</segment>
 </net>
 <net name="+3V3" class="0">
@@
 <segment>
 <pinref part="U1" gate="PORTB_L" pin="PB5"/>
-<wire x1="71.12" y1="-134.62" x2="43.18" y2="-134.62" width="0.1524" layer="91"/>
-<wire x1="43.18" y1="-134.62" x2="43.18" y2="-88.9" width="0.1524" layer="91"/>
-<pinref part="JP2" gate="A" pin="13"/>
-<wire x1="43.18" y1="-88.9" x2="58.42" y2="-88.9" width="0.1524" layer="91"/>
 <pinref part="D2" gate="G$1" pin="A"/>
 <pinref part="X1" gate="G$1" pin="VBUS"/>
-<wire x1="96.52" y1="-38.1" x2="114.3" y2="-38.1" width="0.1524" layer="91"/>
+<wire x1="96.52" y1="-38.1" x2="109.22" y2="-38.1" width="0.1524" layer="91"/>
+<wire x1="109.22" y1="-38.1" x2="114.3" y2="-38.1" width="0.1524" layer="91"/>
 <wire x1="114.3" y1="-38.1" x2="121.92" y2="-38.1" width="0.1524" layer="91"/>
 <wire x1="71.12" y1="-134.62" x2="114.3" y2="-134.62" width="0.1524" layer="91"/>
 <wire x1="114.3" y1="-134.62" x2="114.3" y2="-38.1" width="0.1524" layer="91"/>
-<junction x="71.12" y="-134.62"/>
 <junction x="114.3" y="-38.1"/>
+<pinref part="R13" gate="G$1" pin="2"/>
+<junction x="109.22" y="-38.1"/>
 </segment>
 </net>
@@
 <net name="N$69" class="0">
 <segment>
-<pinref part="TP1" gate="G$1" pin="1"/>
 <pinref part="U1" gate="PORTB_L" pin="PB2"/>
-<wire x1="93.98" y1="-127" x2="71.12" y2="-127" width="0.1524" layer="91"/>
-</segment>
-</net>
+<wire x1="71.12" y1="-127" x2="35.56" y2="-127" width="0.1524" layer="91"/>
+<wire x1="35.56" y1="-127" x2="35.56" y2="-88.9" width="0.1524" layer="91"/>
+<pinref part="JP2" gate="A" pin="13"/>
+<wire x1="35.56" y1="-88.9" x2="58.42" y2="-88.9" width="0.1524" layer="91"/>
+</segment>
+</net>
