File: NintenDAC_AS/nintendac_mini.sch (EAGLE design)
At the start: 21 parts, among them IC1 STM32F10XCXT6, IC3 24C64ST, X1 USB-MICROB

Commit message: continue working on AS
Parts:
- added C1: (no value), backplane:CAP0805
- added LED2: (no value), adafruit:LEDCHIP-LED0805
- added R5, R6, R7: (no value), SparkFun-Passives:RESISTOR0805-RES
- added S2: SWITCH-MOMENTARY-2TURTLE, Adafruit Feather M0 Adalogger:SWITCH-MOMENTARY-2TURTLE
- added TP1, TP10, TP12, TP14, TP16, TP17, TP19, TP2, TP20, TP23, TP8, TP9: TEST-POINTTP_15TH_THRU, pth testpoint:TEST-POINTTP_15TH_THRU
- added TP11, TP13, TP15, TP18, TP21, TP22, TP3, TP4, TP5, TP6, TP7: TEST-POINT3X4, SparkFun-Connectors:TEST-POINT3X4
- JP2: device pinhead:PINHD-2X8 -> pinheadwerew:PINHD-2X8
Connections:
- new net N$10: IC1PORTA_H.PA10, TP1.1
- new net N$11: IC1PORTB_L.PB2, TP4.1
- new net N$12: IC1PORTB_L.PB1, TP5.1
- new net N$13: IC1PORTB_H.PB10, TP3.1
- new net N$14: IC1PORTA_H.PA15, TP6.1
- new net N$15: IC1PORTC.PC13, TP7.1
- new net N$16: IC1PORTC.PC14, TP8.1
- new net N$17: IC1PORTC.PC15, TP9.1
- new net N$18: IC1PORTB_H.PB8, TP10.1
- new net N$19: IC1PORTA_H.PA8, TP11.1
- new net N$20: IC1PORTB_H.PB15, TP12.1
- new net N$21: IC1PORTB_H.PB14, TP13.1
- new net N$22: IC1PORTB_H.PB13, TP14.1
- new net N$23: IC1PORTB_H.PB12, TP15.1
- new net N$24: IC1PORTB_L.PB0, TP16.1
- new net N$25: IC1PORTA_L.PA0, TP18.1
- new net N$26: IC1PORTA_L.PA1, TP17.1
- new net N$27: IC1PORTB_L.PB4, TP20.1
- new net N$28: IC1PORTB_L.PB5, TP19.1
- new net N$29: LED2.C, R7.2
- new net N$5: R6.1, U$3.DOUT, U$4.DIN
- new net N$6: IC1PORTA_H.PA9, TP2.1
- new net SPI1_CS: IC1PORTA_L.PA2, R5.1, U$3.SYNC_N, U$4.SYNC_N
- new net USER_BUTTON: IC1PORTB_H.PB9, S2.1
- new net USER_LED: IC1PORTB_H.PB11, R4.1
- net +3V3: now also C1.1, IC1AN_POWER.VBAT, JP3.3, LED2.A, R5.2, R6.2, U$3.RESET_N, U$4.RESET_N; no longer JP3.6
- net GND: now also C1.2, JP3.6, R7.1, S2.2; no longer JP3.3, R4.1
- net SPI1_MISO: now also TP23.1; no longer U$3.DOUT
- net SPI1_MOSI: now also TP21.1; no longer U$4.DIN
- net SPI1_SCK: now also TP22.1
- net STK: now also IC1PORTA_L.PA3
