File: joyAnalog/joyAnalog.brd (EAGLE design)
At the start: 25 x 37 mm, 50 parts, among them IC1 STM32F10XCXT6, IC3 24C64ST, X1 USB-MICROB

Commit message: finished design, changed name
Parts:
- removed TP23: TEST-POINTTP_15TH_THRU, pth testpoint:TP_15TH
- added R10, R11, R8, R9: (no value), SparkFun-Passives:0805
- moved TP7 12.5 mm to (19.1, 24.5), flipped to the bottom
Connections:
- net +3V3: now also R8.2
- net +5V: now also IC1.2, R9.2
- net GND: now also R11.1, R9.1
- net JC_BAT: now also R10.2
- net N$15: now also R10.1, R11.2; no longer IC1.2
- net SPI1_MISO: now also R8.1; no longer TP23.P$1
Routing:
- net +5V: track 8.53 -> 35.7 mm, vias 0 -> 1
- net +3V3: track 44.1 -> 50.2 mm, vias 0 -> 1
- net JC_BAT: track 3.20 -> 5.74 mm
- net N$15: track 1.34 -> 3.15 mm
- net SPI1_SCK: track 26.7 -> 27.8 mm
- net COLUMN: track 63.4 -> 62.7 mm
Other:
- board text added: "MOSI"
- board text added: "PA0"
- board text added: "PA15"
- board text added: "PB1"
- board text added: "PB10"
- board text added: "PB11"
- board text added: "PB12"
- board text added: "PB14"
- board text added: "PB2"
- board text added: "PB9"
- board text added: "PWR"
- board text added: "RST"
- board text added: "SCK"
- board text added: "dekuNukem 2017"
- board text added: "joyAnalog"

Commit message: firmware update, fixed pcb bug
Parts:
- added R12: (no value), SparkFun-Passives:0805
Connections:
- new net N$30: IC1.2, R12.1
- net +5V: now also R12.2; no longer IC1.2
Routing:
- net +5V: track 35.7 -> 13.0 mm, vias 1 -> 0
- net N$30: track 0.00 -> 21.0 mm, vias 0 -> 1
Changed lines of the file:
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@@
 </element>
 <element name="TP7" library="SparkFun-Connectors" package="PAD.03X.04" value="TEST-POINT3X4" x="19.05" y="24.511" rot="MR0"/>
+<element name="R12" library="SparkFun-Passives" package="0805" value="" x="19.812" y="29.591" rot="MR180"/>
 </elements>
 <signals>
@@
 <wire x1="20.392" y1="30.099" x2="22.606" y2="30.099" width="0.3556" layer="1"/>
 <wire x1="22.606" y1="30.099" x2="23.114" y2="29.591" width="0.3556" layer="1"/>
-<contactref element="IC1" pad="2"/>
 <contactref element="R9" pad="2"/>
 <wire x1="23.114" y1="31.612" x2="23.114" y2="29.591" width="0.2032" layer="16"/>
-<wire x1="16.51" y1="27.432" x2="16.51" y2="18.288" width="0.2032" layer="16"/>
-<wire x1="16.51" y1="18.288" x2="14.097" y2="15.875" width="0.2032" layer="16"/>
-<via x="10.414" y="15.875" extent="1-16" drill="0.508"/>
-<wire x1="14.097" y1="15.875" x2="10.414" y2="15.875" width="0.2032" layer="16"/>
-<wire x1="10.414" y1="15.875" x2="10.196" y2="16.093" width="0.2032" layer="1"/>
-<wire x1="10.196" y1="16.093" x2="10.196" y2="17.217" width="0.2032" layer="1"/>
-<wire x1="23.114" y1="29.591" x2="18.669" y2="29.591" width="0.2032" layer="16"/>
-<wire x1="18.669" y1="29.591" x2="16.51" y2="27.432" width="0.2032" layer="16"/>
+<contactref element="R12" pad="2"/>
+<wire x1="20.712" y1="29.591" x2="23.114" y2="29.591" width="0.2032" layer="16"/>
 </signal>
 <signal name="N$3">
@@
 <wire x1="19.05" y1="24.511" x2="20.574" y2="24.511" width="0.2032" layer="16"/>
 </signal>
+<signal name="N$30">
+<contactref element="IC1" pad="2"/>
+<contactref element="R12" pad="1"/>
+<wire x1="18.912" y1="29.591" x2="16.383" y2="27.062" width="0.2032" layer="16"/>
+<wire x1="16.383" y1="27.062" x2="16.383" y2="17.78" width="0.2032" layer="16"/>
+<wire x1="16.383" y1="17.78" x2="14.478" y2="15.875" width="0.2032" layer="16"/>
+<wire x1="14.478" y1="15.875" x2="10.414" y2="15.875" width="0.2032" layer="16"/>
+<via x="10.414" y="15.875" extent="1-16" drill="0.5"/>
+<wire x1="10.414" y1="15.875" x2="10.196" y2="16.093" width="0.2032" layer="1"/>
+<wire x1="10.196" y1="16.093" x2="10.196" y2="17.217" width="0.2032" layer="1"/>
+</signal>
 </signals>
